File: HW/Microwavino.sch (KiCad schematic (older format))
At the start: 56 parts, among them P1 SMA, P2 SMA, P3 SMA, P4 SMA, U1 MIC5366, U2 MCP1824T, U3 MCP1824T, U4 MCP1824T, U5 ASTXR-12-19.200MHz, U6 MAX2871, U7 Teensy3.2

Commit message: before placement
Parts:
- D1: footprint (none) -> LEDs:LED_0603
