File: HW/Microwavino.sch (KiCad schematic (older format))
At the start: 52 parts, among them P1 SMA, U1 MIC5366, U2 MCP1824T, U3 MCP1824T, U4 MCP1824T, U5 ASTXR-12-19.200MHz, U6 MAX2871, U7 Teensy3.2

Commit message: drc pass
Connections:
- net GND: now also U7.10 (8_TX3_DIN), U7.11 (9_RX2_CS_PWM), U7.23 (16_A2_SCL0_Touch), U7.24 (17_A3_SDA0_Touch)
- net MUXOUT: now also U7.14 (12_DIN); no longer U7.8 (6_PWM)
- net RFOUT_EN: now also U7.8 (6_PWM); no longer U7.9 (7_RX3_DOUT)
- no-connect marks 48 -> 44
Changed lines of the file:
@@
 Text Label 12950 4450 0    60   ~ 0
 LD
-Text Label 9850 2650 2    60   ~ 0
+Text Label 9850 2550 2    60   ~ 0
 RFOUT_EN
-Text Label 9850 2550 2    60   ~ 0
+Text Label 9850 3150 2    60   ~ 0
 MUXOUT
 NoConn ~ 12400 2150
@@
 NoConn ~ 12400 4250
 NoConn ~ 12400 4350
-NoConn ~ 10400 3150
 NoConn ~ 10400 3350
 NoConn ~ 10400 3450
 NoConn ~ 10400 3550
 NoConn ~ 10400 3650
-NoConn ~ 10400 4150
 NoConn ~ 10400 4250
 NoConn ~ 10400 4350
 NoConn ~ 10400 4450
-NoConn ~ 10400 4050
 NoConn ~ 10400 3850
 NoConn ~ 10400 3950
@@
 	9850 2450 10400 2450
 Wire Wire Line
+	9850 3150 10400 3150
+Wire Wire Line
 	9850 2550 10400 2550
-Wire Wire Line
-	9850 2650 10400 2650
 Wire Wire Line
 	12950 4450 12400 4450
@@
 Wire Wire Line
 	12700 7450 12700 7250
-NoConn ~ 10400 2850
 NoConn ~ 10400 2950
 NoConn ~ 10400 3250
-NoConn ~ 10400 2750
 Wire Wire Line
 	7450 6000 7400 6000
@@
 	7450 5550 7650 5550
 Connection ~ 7450 5550
+$Comp
+L GND #PWR039
+U 1 1 59B68B65
+P 10050 2850
+F 0 "#PWR039" H 10050 2600 50  0001 C CNN
+F 1 "GND" H 10050 2700 50  0000 C CNN
+F 2 "" H 10050 2850 60  0000 C CNN
+F 3 "" H 10050 2850 60  0000 C CNN
+	1    10050 2850
+	0    1    1    0
+$EndComp
+Wire Wire Line
+	10050 2850 10400 2850
+$Comp
+L GND #PWR040
+U 1 1 59B68BA2
+P 10050 4150
+F 0 "#PWR040" H 10050 3900 50  0001 C CNN
+F 1 "GND" H 10050 4000 50  0000 C CNN
+F 2 "" H 10050 4150 60  0000 C CNN
+F 3 "" H 10050 4150 60  0000 C CNN
+	1    10050 4150
+	0    1    1    0
+$EndComp
+Wire Wire Line
+	10050 4150 10400 4150
+Wire Wire Line
+	10400 4050 10300 4050
+Wire Wire Line
+	10300 4050 10300 4150
+Connection ~ 10300 4150
+Wire Wire Line
+	10400 2750 10300 2750
+Wire Wire Line
+	10300 2750 10300 2850
+Connection ~ 10300 2850
+NoConn ~ 10400 2650
 $EndSCHEMATC

Commit message: added footprint SOT-323-70-sc-5
Parts:
- U1: footprint VNA:SOT-23-5 -> VNA:SOT-353_SC-70-5
Changed lines of the file:
@@
 LIBS:valves
 LIBS:vna-cache
-LIBS:teensy
 LIBS:Microwavino-cache
 EELAYER 25 0
@@
 F 0 "U1" H 3250 5800 60  0000 C CNN
 F 1 "MIC5366" H 3100 6200 60  0000 C CNN
-F 2 "VNA:SOT-23-5" H 3050 5850 60  0001 C CNN
+F 2 "VNA:SOT-353_SC-70-5" H 3050 5850 60  0001 C CNN
 F 3 "" H 3050 5850 60  0000 C CNN
 	1    3100 6000

Commit message: added sw and wiki
Other:
- note added: "Replaced because RS doesn't have them:\nMIC5366 with TLV70018 \nASTXR-12-19.2MHz with ASD3-24.000MHz-EC"
Changed lines of the file:
@@
 Connection ~ 10300 2850
 NoConn ~ 10400 2650
+Text Notes 2030 6830 0    60   ~ 0
+Replaced because RS doesn't have them:\nMIC5366 with TLV70018 \nASTXR-12-19.2MHz with ASD3-24.000MHz-EC
 $EndSCHEMATC
